File: picow_vga_sd_aud.kicad_sch (KiCad schematic)
At the start: 71 parts, among them J10 Micro_SD_Card, J2 AudioJack3, J3 Micro_SD_Card, J4 L77HDE15SD1CH4F, J7 Conn_02x03_Odd_Even, J8 TSW-102-07-G-S, J9 Mini-DIN-6, SW1 SW_Push, SW2 SW_Push, SW3 SW_Push, SW4 SW_Push, U1 TLV70033_SOT23-5, U10 ER_OLEDM0.91_1x-I2C, U11 TL431DBZ, U2 PicoW, U3 NC7WZ16P6X

Commit message: Fix LCSC placement
Parts:
- R26: LCSC (none) -> C25108
Changed lines of the file:
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@@
 					(size 1.27 1.27)
 				)
-					(property "LCSC" "C25108"
+			)
+		)
+		(property "LCSC" "C25108"
 			(at 0 0 0)
 			(hide yes)
@@
 			)
 		)
-)
-		)
 		(property "Footprint" "Resistor_SMD:R_0805_2012Metric"

Commit message: Fix LCSC placement
Parts:
- R27: LCSC (none) -> C11702
Changed lines of the file:
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@@
 					(size 1.27 1.27)
 				)
-					(property "LCSC" "C11702"
+			)
+		)
+		(property "LCSC" "C11702"
 			(at 0 0 0)
 			(hide yes)
@@
 			)
 		)
-)
-		)
 		(property "Footprint" "Resistor_SMD:R_0805_2012Metric"
