File: picow_vga_sd_aud.kicad_sch (KiCad schematic)
At the start: 64 parts, among them J10 Micro_SD_Card, J2 AudioJack3, J3 Micro_SD_Card, J4 L77HDE15SD1CH4F, J7 Conn_02x03_Odd_Even, SW1 SW_Push, SW2 SW_Push, SW3 SW_Push, SW4 SW_Push, U1 TLV70033_SOT23-5, U10 ER_OLEDM0.91_1x-I2C, U2 PicoW, U3 NC7WZ16P6X

Commit message: Últimos cambios: referencias Arial, clearances net classes, vias 0.6mm
Parts:
- added J8: TSW-102-07-G-S, RaspberryPI PicoW:samtec_tsw-102-07-g-s, symbol RPI_DB:Connectors | Pin_Headers/RP-01JV5X-LY21H5
Connections:
- net +3.3VA is gone; now on net +3V3: C2.1, C4.1, R42.2, R43.2, U1.5 (OUT), U10.2 (VCC), U3.5 (VCC)
- net GND: now also J8.2 (Pin_2)
- net VSYS: now also J8.1 (Pin_1)

Commit message: Update schematics and PCB
Parts:
- added C27: 1u, Capacitor_SMD:C_0805_2012Metric, symbol Device:C
- added J9: Mini-DIN-6, kiC:TE_5749180-1, symbol Connector:Mini-DIN-6
- added R46, R47, R48: 1k, Resistor_SMD:R_0805_2012Metric, symbol Device:R
- added U11: TL431DBZ, Package_TO_SOT_SMD:SOT-23, symbol Reference_Voltage:TL431DBZ
- J3, R23, R24, R9, U2: now left out of the parts list
Connections:
- net +3V3: now also R48.1; no longer C2.1, C4.1, U1.5 (OUT), U3.5 (VCC)
- net GND: now also C27.2, J9.3, U11.3 (A)
- net GPIO26: now also J9.1
- net GPIO27: now also J9.5
- net GPIO29: now also U2.35 (ADC_VREF), R46.2
- net VSYS: now also J9.4
- new net: C27.1, R46.1, R47.2
- new net: R48.2, U11.1 (K)
- new net: R47.1, U11.2 (REF)
- new net +3.3VA: C2.1, C4.1, U1.5 (OUT), U3.5 (VCC)
- no-connect marks 9 -> 10
Other:
- title: RPI-PWVSA    VGA, SD Card & Audio Demo Board for Pico W -> VGA, SD Card

Commit message: Import LCSC from CSV
Parts:
- C1, C14, C19, C2, C27, C4, C7: LCSC (none) -> C28233
- C15: LCSC (none) -> C107110
- C8: LCSC (none) -> C48587228
- D1: LCSC (none) -> C2297
- J10: LCSC (none) -> C125617
- J3: LCSC (none) -> C91144
- R10, R11: LCSC (none) -> C17477
- R15, R16, R27, R28, R29, R30, R31, R32, R33, R34, R35, R36, R39, R42: LCSC (none) -> C17520
- R18, R19, R20, R38, R40: LCSC (none) -> C17414
- R21, R43, R44, R45, R46, R47, R48: LCSC (none) -> C17673
- R22, R23: LCSC (none) -> C2933393
- R24, R8, R9: LCSC (none) -> C17513
- SW1: LCSC (none) -> C92584
- SW3, SW4: LCSC (none) -> C83916
- U1: LCSC (none) -> C5366877
- U10: LCSC (none) -> C97521
- U11: LCSC (none) -> C220623

Commit message: Update files
Parts:
- C1, C2, C27: LCSC C28233 -> C1779
- C14: LCSC C28233 -> (none)
- C15: LCSC C107110 -> (none)
- C19: LCSC C28233 -> C15850
- C8: LCSC C48587228 -> C28233
- J7, U10: now left out of the parts list
- R15, R28, R29, R30, R31, R33, R34, R35, R36, R39: LCSC C17520 -> (none)
- R17: LCSC (none) -> C17520
- R18, R19: LCSC C17414 -> C17520
- R20: LCSC C17414 -> C17673
- R22: LCSC C2933393 -> C17673
- R23: LCSC C2933393 -> C17414
- R24: LCSC C17513 -> C17414
- R27, R32: LCSC C17520 -> C17673
- R37: LCSC (none) -> C17673
- R38, R40: LCSC C17414 -> (none)
- R43, R44, R45: LCSC C17673 -> C17520
- R8: LCSC C17513 -> (none)
Changed lines of the file:
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@@
 			)
 		)
-		(property "LCSC" "C17520"
+		(property "LCSC" "C17673"
 			(at 311.15 36.83 90)
 			(hide yes)
@@
 			)
 		)
-		(property "LCSC" "C17520"
+		(property "LCSC" ""
 			(at 311.15 41.91 90)
 			(hide yes)
@@
 			)
 		)
-		(property "LCSC" "C17520"
+		(property "LCSC" ""
 			(at 311.15 46.99 90)
 			(hide yes)
@@
 			)
 		)
-		(property "LCSC" "C17520"
+		(property "LCSC" ""
 			(at 311.15 52.07 90)
 			(hide yes)
@@
 			)
 		)
-		(property "LCSC" "C17414"
+		(property "LCSC" "C17673"
 			(at 281.94 45.72 90)
 			(hide yes)
@@
 			)
 		)
-		(property "LCSC" "C17520"
+		(property "LCSC" ""
 			(at 311.15 68.58 90)
 			(hide yes)
@@
 			)
 		)
-		(property "LCSC" "C17520"
+		(property "LCSC" "C17673"
 			(at 311.15 73.66 90)
 			(hide yes)
@@
 			)
 		)
-		(property "LCSC" "C17520"
+		(property "LCSC" ""
 			(at 311.15 78.74 90)
 			(hide yes)
@@
 			)
 		)
-		(property "LCSC" "C17520"
+		(property "LCSC" ""
 			(at 311.15 88.9 90)
 			(hide yes)
@@
 			)
 		)
-		(property "LCSC" "C17520"
+		(property "LCSC" ""
 			(at 311.15 105.41 90)
 			(hide yes)
@@
 			)
 		)
-		(property "LCSC" ""
+		(property "LCSC" "C17673"
 			(at 311.15 110.49 90)
 			(hide yes)
@@
 			)
 		)
-		(property "LCSC" "C17414"
+		(property "LCSC" ""
 			(at 311.15 115.57 90)
 			(hide yes)
@@
 			)
 		)
-		(property "LCSC" "C17520"
+		(property "LCSC" ""
 			(at 311.15 120.65 90)
 			(hide yes)
@@
 			)
 		)
-		(property "LCSC" "C17414"
+		(property "LCSC" ""
 			(at 311.15 125.73 90)
 			(hide yes)
@@
 			)
 		)
-		(property "LCSC" "C2933393"
+		(property "LCSC" "C17673"
 			(at 281.94 119.38 90)
 			(hide yes)
@@
 			)
 		)
-		(property "LCSC" "C17520"
+		(property "LCSC" ""
 			(at 311.15 83.82 90)
 			(hide yes)
@@
 			)
 		)
-		(property "LCSC" "C28233"
+		(property "LCSC" ""
 			(at 168.91 232.41 90)
 			(hide yes)
@@
 			)
 		)
-		(property "LCSC" "C28233"
+		(property "LCSC" "C15850"
 			(at 356.87 143.51 0)
 			(hide yes)
@@
 			)
 		)
-		(property "LCSC" "C48587228"
+		(property "LCSC" "C28233"
 			(at 148.59 260.35 0)
 			(hide yes)
@@
 			)
 		)
-		(property "LCSC" "C107110"
+		(property "LCSC" ""
 			(at 168.91 254 90)
 			(hide yes)
@@
 			)
 		)
-		(property "LCSC" "C17513"
+		(property "LCSC" ""
 			(at 176.53 260.35 0)
 			(hide yes)
@@
 			)
 		)
-		(property "LCSC" "C17513"
+		(property "LCSC" "C17414"
 			(at 334.01 144.78 0)
 			(hide yes)
@@
 			)
 		)
-		(property "LCSC" "C2933393"
+		(property "LCSC" "C17414"
 			(at 326.39 144.78 0)
 			(hide yes)
@@
 		(body_style 1)
 		(exclude_from_sim no)
-		(in_bom yes)
+		(in_bom no)
 		(on_board yes)
 		(in_pos_files yes)
@@
 			)
 		)
-		(property "LCSC" "C28233"
+		(property "LCSC" "C1779"
 			(at 168.91 45.72 0)
 			(hide yes)
@@
 			)
 		)
-		(property "LCSC" "C28233"
+		(property "LCSC" "C1779"
 			(at 199.39 45.72 0)
 			(hide yes)
@@
 			)
 		)
-		(property "LCSC" "C17673"
+		(property "LCSC" "C17520"
 			(at 189.23 176.53 0)
 			(hide yes)
@@
 			)
 		)
-		(property "LCSC" "C28233"
+		(property "LCSC" "C1779"
 			(at 160.02 101.6 0)
 			(hide yes)
@@
 		(body_style 1)
 		(exclude_from_sim no)
-		(in_bom yes)
+		(in_bom no)
 		(on_board yes)
 		(in_pos_files yes)
@@
 			)
 		)
-		(property "LCSC" ""
+		(property "LCSC" "C17520"
 			(at 303.53 213.36 0)
 			(hide yes)
@@
 			)
 		)
-		(property "LCSC" "C17673"
+		(property "LCSC" "C17520"
 			(at 318.77 213.36 0)
 			(hide yes)
@@
 			)
 		)
-		(property "LCSC" "C17414"
+		(property "LCSC" "C17520"
 			(at 295.91 213.36 0)
 			(hide yes)
@@
 			)
 		)
-		(property "LCSC" "C17414"
+		(property "LCSC" "C17520"
 			(at 288.29 213.36 0)
 			(hide yes)
@@
 			)
 		)
-		(property "LCSC" "C17673"
+		(property "LCSC" "C17520"
 			(at 321.31 238.76 0)
 			(hide yes)
@@
 			)
 		)
-		(property "LCSC" "C17520"
+		(property "LCSC" ""
 			(at 255.27 233.68 0)
 			(hide yes)
