File: pico.kicad_sch (KiCad schematic)
At the start: 34 parts, among them J1 10103594-0001LF, J5 TSW-102-07-G-S, SW5 SW_boot, U4 NCP1117ST33T3G, U5 W25Q128JVSIQ, U6 RP2040, U7 W25Q128JVSIQ, X1 12MHz

Commit message: Update files
Parts:
- C10, C11, C24: footprint Capacitor_SMD:C_0603_1608Metric -> Capacitor_SMD:C_0402_1005Metric; LCSC (none) -> C1525
- C12, C16, C18, C20, C21, C22, C23: LCSC (none) -> C28233
- C13, C17: footprint Capacitor_SMD:C_0603_1608Metric -> Capacitor_SMD:C_0805_2012Metric; LCSC (none) -> C1779
- C25, C6: LCSC (none) -> C15850
- C3, C5: LCSC (none) -> C107110
- C9: footprint Capacitor_SMD:C_0603_1608Metric -> Capacitor_SMD:C_0805_2012Metric; LCSC (none) -> C15850
- L1: value 100mH -> 100uH; footprint Resistor_SMD:R_2512_6332Metric -> Inductor_SMD:L_1206_3216Metric; LCSC (none) -> C74489
- R12, R41: LCSC (none) -> C17513
- R13, R14: LCSC (none) -> C2933393
- R5: LCSC (none) -> C17673
- R6: LCSC (none) -> C17414
- U6: now left out of the parts list
