File: picow_vga_sd_aud.kicad_pcb (KiCad board)
At the start: 4 copper layers, 74.4 x 65.8 mm, 108 parts, among them J1 10103594-0001LF, J10 Micro_SD_Card, J2 AudioJack3, J3 Micro_SD_Card, J4 L77HDE15SD1CH4F, J5 TSW-102-07-G-S, J6 Conn_01x18_Pin, J7 Conn_02x03_Odd_Even, J8 TSW-102-07-G-S, J9 Mini-DIN-6, SW1 SW_Push, SW2 SW_Push, SW3 SW_Push, SW4 SW_Push, SW5 SW_boot, U1 TLV70033_SOT23-5, U10 ER_OLEDM0.91_1x-I2C, U11 TL431DBZ, U2 PicoW, U3 NC7WZ16P6X, U4 NCP1117ST33T3G, U5 W25Q128JVSIQ, U6 RP2040, U7 W25Q128JVSIQ, U8 TXS0108, U9 TXS0108, X1 12MHz

Commit message: Update files
Parts:
- C10, C11, C24: footprint Capacitor_SMD:C_0603_1608Metric -> Capacitor_SMD:C_0402_1005Metric
- C13, C17, C9: footprint Capacitor_SMD:C_0603_1608Metric -> Capacitor_SMD:C_0805_2012Metric
- L1: value 100mH -> 100uH; footprint Resistor_SMD:R_2512_6332Metric -> Inductor_SMD:L_1206_3216Metric

Commit message: update . files
Parts:
- moved C4 0.77 mm to (144.8, 79.2)
- moved C13 0.33 mm to (136.0, 72.8)
Routing:
- net GND: track 506.5 -> 561.4 mm, vias 338 -> 515
- net VBUS: track 135.3 -> 137.7 mm
- net Net-(U4-IN): track 25.5 -> 26.9 mm
- net +1V1: track 21.3 -> 22.6 mm
- removed copper zone on In1.Cu, net GND
- removed copper zone on In2.Cu, net GND
Other:
- copper layers 4 -> 2
